File: eagle/ewod-1x4.sch (EAGLE design)
At the start: 19 parts

Commit message: redo to 50x50mm
Parts:
- removed 3.3V: VREG, nonolith:VREG
- removed C10: 1uF, nonolith:CAP_CERAMIC0603
- removed C11: .1uF, nonolith:CAP_CERAMIC0603
- removed C12: .01uF, nonolith:CAP_CERAMIC0603
- removed PORTE: (no value), nonolith:HEADER-1X62MM
- removed PROGX: (no value), nonolith:HEADER-2X3
- removed XM1: (no value), nonolith:ATXMEGAXXA4U-MH
- added ATXMEGA32A4U: (no value), nonolith:ATXMEGAXXA4U-AU
- added C1, C2, C5: (no value), nonolith:CAP_CERAMIC0603
- added JP1: (no value), nonolith:HEADER-2X3
- added U$10: MCP1700, nonolith:MCP1700
- added U$12: M19, SparkFun:M19
- R1: value 120o -> (none)
Connections:
- removed net 3.3V: 3.3V.VO, C10.P$2, C11.P$2, C12.P$2, PROGX.2, XM1.AVCC, XM1.VCC@1, XM1.VCC@2, XM1.VCC@3
- removed net 5V: 3.3V.VIN, CN1.VBUS, PORTE.1
- removed net ADCA: RN3D.2, RN4D.1, XM1.PA0/ADC0/AREFA
- removed net ADCB: RN3C.2, RN4C.1, XM1.PA1/ADC1
- removed net ADCC: RN3B.2, RN4B.1, XM1.PA2/ADC2
- removed net ADCD: RN3A.2, RN4A.1, XM1.PA3/ADC3
- removed net BOOTLOAD: PROGX.4, XM1.PR0/XTAL2
- removed net OC0A: RN1A.2, XM1.PC0/OC0A/SDA
- removed net OC0B: RN1B.2, XM1.PC1/OC0B/XCK0/SCL
- removed net OC0C: RN1C.2, XM1.PC2/OC0C/RXD0
- removed net OC0D: RN1D.2, XM1.PC3/OC0D/TXD0
- removed net PR1: R1.1, XM1.PR1/XTAL1
- removed net PR1-P: LED1.A, R1.2
- new net N$1: LED1.C, R1.1
- new net PA0: ATXMEGA32A4U.PA0/ADC0/AREFA, RN3D.2, RN4D.1
- new net PA1: ATXMEGA32A4U.PA1/ADC1, RN3C.2, RN4C.1
- new net PA2: ATXMEGA32A4U.PA2/ADC2, RN3B.2, RN4B.1
- new net PA3: ATXMEGA32A4U.PA3/ADC3, RN3A.2, RN4A.1
- new net PA4: ATXMEGA32A4U.PA4/ADC4
- new net PA5: ATXMEGA32A4U.PA5/ADC5
- new net PA6: ATXMEGA32A4U.PA6/ADC6
- new net PA7: ATXMEGA32A4U.PA7/ADC7
- new net PB0: ATXMEGA32A4U.PB0/ADC8/AREFB
- new net PB1: ATXMEGA32A4U.PB1/ADC9
- new net PB2: ATXMEGA32A4U.PB2/ADC10/DAC0
- new net PB3: ATXMEGA32A4U.PB3/ADC11/DAC1
- new net PC0: ATXMEGA32A4U.PC0/OC0A/SDA
- new net PC1: ATXMEGA32A4U.PC1/OC0B/XCK0/SCL
- new net PC2: ATXMEGA32A4U.PC2/OC0C/RXD0, U$12.19
- new net PC3: ATXMEGA32A4U.PC3/OC0D/TXD0, U$12.18
- new net PC4: ATXMEGA32A4U.PC4/OC1A/#SS, RN1D.2, U$12.17
- new net PC5: ATXMEGA32A4U.PC5/OC1B/MOSI/XCK1, RN1C.2, U$12.16
- new net PC6: ATXMEGA32A4U.PC6/MISO/RXD1, RN1B.2, U$12.15
- new net PC7: ATXMEGA32A4U.PC7/SCK/TXD1/CLKO/EVO, RN1A.2, U$12.14
- new net PD0: ATXMEGA32A4U.OC0A/PD0, U$12.13
- new net PD1: ATXMEGA32A4U.OC0B/XCK0/PD1, U$12.12
- new net PD2: ATXMEGA32A4U.OC0C/RXD0/PD2, U$12.11
- new net PD3: ATXMEGA32A4U.OC0D/TXD0/PD3, U$12.10
- new net PD4: ATXMEGA32A4U.SS/PD4, U$12.9
- new net PD5: ATXMEGA32A4U.XCK1/MOSI/PD5, U$12.8
- new net VCC: ATXMEGA32A4U.AVCC, ATXMEGA32A4U.VCC@1, ATXMEGA32A4U.VCC@2, ATXMEGA32A4U.VCC@3, C1.P$1, C2.P$1, JP1.2, U$10.VO, U$12.2
- new net VUSB: C5.P$1, CN1.VBUS, U$10.V+
- net GND: now also ATXMEGA32A4U.GND@1, ATXMEGA32A4U.GND@2, ATXMEGA32A4U.GND@3, ATXMEGA32A4U.GND@4, C1.P$2, C2.P$2, C5.P$2, JP1.6, R1.2, U$10.GND, U$12.1, U$12.3; no longer 3.3V.GND, C10.P$1, C11.P$1, C12.P$1, LED1.C, PORTE.6, PROGX.6, XM1.GND@1, XM1.GND@2, XM1.GND@3, XM1.GND@4
- net PDI-CLK: now also ATXMEGA32A4U.RESET/PDI-CLK, JP1.5; no longer PROGX.5, XM1.RESET/PDI-CLK
- net PDI-DATA: now also ATXMEGA32A4U.PDI-DATA, JP1.1; no longer PROGX.1, XM1.PDI-DATA
- net PE0: now also ATXMEGA32A4U.OC0A/SDA/PE0, U$12.7; no longer PORTE.2, XM1.OC0A/SDA/PE0
- net PE1: now also ATXMEGA32A4U.XCK0/OC0B/SCL/PE1, U$12.6; no longer PORTE.3, XM1.XCK0/OC0B/SCL/PE1
- net PE2: now also ATXMEGA32A4U.RXD0/OC0C/PE2, LED1.A, U$12.5; no longer PORTE.4, XM1.RXD0/OC0C/PE2
- net PE3: now also ATXMEGA32A4U.TXD0/OC0D/PE3, U$12.4; no longer PORTE.5, XM1.TXD0/OC0D/PE3
- net USB+: now also ATXMEGA32A4U.TXD1/USB+/PD7; no longer XM1.TXD1/USB+/PD7
- net USB-: now also ATXMEGA32A4U.RXD1/MISO/USB-/PD6; no longer XM1.RXD1/MISO/USB-/PD6
